File: Hardware/BMS/DroneBMS.kicad_sch (KiCad schematic)
At the start: 38 parts, among them J1 BattLevel (ADC), J2 BattLevel (ADC), U1 LMR51430, U2 AMS1117-3.3

Commit message: Updated Pcb Footprints
Parts:
- L1: footprint Inductor_SMD:L_Bourns-SRN6028 -> Custom_Footprints:IND_VSAB0630-4R7M
Changed lines of the file:
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@@
 			)
 		)
-		(property "Footprint" "Inductor_SMD:L_Bourns-SRN6028"
+		(property "Footprint" "Custom_Footprints:IND_VSAB0630-4R7M"
 			(at 138.43 55.88 0)
 			(effects
